File: Hardware/ESP8266-Thing-Dev-4H.sch (EAGLE design)
At the start: 70 parts, among them J1 U.FL, Q1 MMBT2222A, Q2 MMBT2222A, U1 AP2112K-3.3V, U2 ESP8266, U3 AT25SF041-SOIC8, U4 FTS31XS-U, Y1 26MHz

Commit message: Updating libraries, increasing width of 4H logo lines.
Parts:
- C1: device SparkFun-Capacitors:10UF-6.3V-20%(0603) -> SparkFun-Capacitors:10UF-0603-6.3V-20%
- C10, C12, C14, C2, C8: device SparkFun-Capacitors:0.1UF-25V(+80/-20%)(0603) -> SparkFun-Capacitors:0.1UF-0603-25V-(+80/-20%)
- C11, C9: device SparkFun-Capacitors:47PF-50V-5%(0603) -> SparkFun-Capacitors:47PF-0603-50V-5%
- C13: device SparkFun-Capacitors:10UF-16V-10%(TANT) -> SparkFun-Capacitors:10UF-POLAR-EIA3216-16V-10%(TANT)
- C3, C4: device SparkFun-Capacitors:10PF-50V-5%(0603) -> SparkFun-Capacitors:10PF-0603-50V-5%
- C5: device SparkFun-Capacitors:1.0UF-25V-+80/-20(0805) -> SparkFun-Capacitors:1.0UF-0805-25V-(+80/-20%)
- C6: device SparkFun-Capacitors:2.2UF-10V-20%(0603) -> SparkFun-Capacitors:2.2UF-0603-10V-20%
- C7: value 5.6pF -> 5.6PF; device SparkFun-Capacitors:CAP0603-CAP -> SparkFun-Capacitors:5.6PF-0603-50V-5%
- D1: value BAT20J -> 1A/23V/620mV
- E1: value ANTENNATRACE -> ANTENNA-GROUNDEDTRACE-25.7MM; device SparkFun-RF:ANTENNATRACE -> SparkFun-RF:ANTENNA-GROUNDEDTRACE-25.7MM
- Q1, Q2: value MMBT2222A -> 600mA/40V; device SparkFun-DiscreteSemi:TRANSISTOR_NPNMMBT2222A -> SparkFun-DiscreteSemi:TRANS_NPN-MMBT2222AL
- R1: device SparkFun-Resistors:12KOHM-1/10W-1%(0603) -> SparkFun-Resistors:12KOHM-0603-1/10W-1%
- R10, R11, R14, R17, R2, R5, R9: value 10K -> 10k; device SparkFun-Resistors:10KOHM1/10W1%(0603)0603 -> SparkFun-Resistors:10KOHM-0603-1/10W-1%
- R12, R13, R15, R16: value 1K -> 1k; device SparkFun-Resistors:1KOHM-1/10W-1%(0603) -> SparkFun-Resistors:1KOHM-0603-1/10W-1%
- R3, R4, R6: device SparkFun-Resistors:200OHM1/10W1%(0603) -> SparkFun-Resistors:200OHM-0603-1/10W-1%
- R7, R8: device SparkFun-Resistors:27OHM1/10W1%(0603)0603-RES -> SparkFun-Resistors:27OHM-0603-1/10W-1%
- S1: device SparkFun-Electromechanical:SWITCH-SPDT-SMD-A -> SparkFun-Switches:SWITCH-SPDT-SMD-RIGHT-ANGLE
- STANDOFF1, STANDOFF2, STANDOFF3, STANDOFF4: device SparkFun-Electromechanical:STAND-OFF -> SparkFun-Hardware:STAND-OFF
- U2: device esp8266-development-board:ESP8266 -> SparkFun-RF:ESP8266
